File: electronic/MecProInverter/_autosave-power.kicad_sch (KiCad schematic)
At the start: 57 parts, among them J3 Conn_01x02, J4 Screw_Terminal_01x08, K2 RT314A12, Q1 DMN3404L, U3 IKCM20L60GA, U4 LVE2560E, U5 TPS563201DDCR, U8 TLA2528IRTER

Commit message: electronic
-Control: Added Temp, Fan,
Parts:
- added R35: R, symbol Device:R
Connections:
- net +3.3V: now also C38.2, C39.1, U8.10 (DVDD), U8.7 (AVDD)
- net GND: now also R39.2
- net at R39.1, U8.11 (ADDR): now also R35.2
- net at U8.8 (DECAP): now also R35.1
Other:
- moved on the sheet: C38, C39
