File: electronic/MecProInverter/power.kicad_sch (KiCad schematic)
At the start: 57 parts, among them J3 Conn_01x02, J4 Screw_Terminal_01x08, K2 RT314A12, Q1 DMN3404L, U3 IKCM20L60GA, U4 LVE2560E, U5 TPS563201DDCR, U8 TLA2528IRTER

Commit message: electronic
Added: current sensor
Parts:
- added C26, C41, C42, C43, C44, C45: C, symbol Device:C
- added R35: 999m, symbol Device:R
- added R40, R41: R, symbol Device:R
- added U10, U12, U9: ACS722xLCTR-40AB, Package_SO:SOIC-8_3.9x4.9mm_P1.27mm, symbol Sensor_Current:ACS722xLCTR-40AB
- C1, C2, C3, C4: footprint (none) -> footprints:ESMQ351VSN102MA50S
- J4: footprint (none) -> Connector_Phoenix_MC_HighVoltage:PhoenixContact_MCV_1,5_8-G-5.08_1x08_P5.08mm_Vertical
- R39: value R -> 33k
- renumbered U3 to U13
Connections:
- net +3.3V: now also C38.2, C39.1, U8.10 (DVDD), U8.7 (AVDD), C26.2, C43.2, C45.2, U10.8 (VCC), U12.8 (VCC), U9.8 (VCC)
- net AC_L: now also R40.1
- net CURRENT_AC: now also C41.2, U10.7 (VIOUT)
- net GND: now also R39.2, C26.1, C41.1, C42.1, C43.1, C44.1, C45.1, R41.2, U10.5 (GND), U10.6 (BW_SEL), U12.5 (GND), U12.6 (BW_SEL), U9.5 (GND), U9.6 (BW_SEL)
- net U: now also U12.3 (IP-), U12.4 (IP-); no longer U13.22 (U)
- net W: now also U9.3 (IP-), U9.4 (IP-); no longer U13.20 (W)
- net at R39.1, U8.11 (ADDR): now also R35.2
- net at U8.2 (AIN3/GPIO3): now also C42.2, U12.7 (VIOUT)
- net at U8.3 (AIN4/GPIO4): now also C44.2, U9.7 (VIOUT)
- net at U8.6 (AIN7/GPIO7): now also R40.2, R41.1
- net at U8.8 (DECAP): now also R35.1
- net at K2.14, R1.2: now also U10.1 (IP+), U10.2 (IP+); no longer U4.2 (~Phase)
- new net: U10.3 (IP-), U10.4 (IP-), U4.2 (~Phase)
- new net: U13.20 (W), U9.1 (IP+), U9.2 (IP+)
- new net: U12.1 (IP+), U12.2 (IP+), U13.22 (U)
Other:
- moved on the sheet: C1, C10, C11, C12, C13, C14, C15, C16, C17, C18, C19, C2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

Commit message: Electronic
Currentsensor updated
Power structure updated
Parts:
- removed J3: Conn_01x02, symbol Connector_Generic:Conn_01x02
- removed U10, U12, U9: ACS722xLCTR-40AB, Package_SO:SOIC-8_3.9x4.9mm_P1.27mm, symbol Sensor_Current:ACS722xLCTR-40AB
- added D6: D, symbol Device:D
- added R43, R44, R45: 100, symbol Device:R
- added R49: 33k, symbol Device:R
- added R50: 66k, symbol Device:R
- added U10, U11, U9: CC6904SO-30A, footprint:SOP-8_L4.9-W3.9-P1.27-LS6.0-BL, symbol CC6904SO-30A:CC6904SO-30A
- added U14: DMP3098L-7, footprint:SOT-23_L2.9-W1.3-P1.90-LS2.4-BR, symbol DMP3098L-7:DMP3098L-7
- C26, C43, C45: value C -> 100nF
- C41, C42, C44: value C -> 0.1nF
Connections:
- net +15V: now also D6.2 (A), R50.1
- net +3.3V: now also U10.8 (VCC), U11.8 (VCC), U9.8 (VCC)
- net CURRENT_AC: now also R43.2
- net GND: now also R49.2, U10.5 (GND), U11.5 (GND), U9.5 (GND)
- net U: now also U10.4 (IP-)
- net VS: now also D6.1 (K), U14.3 (D)
- net W: now also U11.4 (IP-)
- net at C42.2, U8.2 (AIN3/GPIO3): now also R44.2
- net at C44.2, U8.3 (AIN4/GPIO4): now also R45.2
- net at K2.14, R1.2: now also U9.1 (IP+)
- net at U4.2 (~Phase): now also U9.4 (IP-)
- net at U13.20 (W): now also U11.1 (IP+)
- net at U13.22 (U): now also U10.1 (IP+)
- new net: R44.1, U10.7 (OUT)
- new net: R43.1, U9.7 (OUT)
- new net: R45.1, U11.7 (OUT)
- new net: R49.1, R50.2, U14.1 (G)
- new net +5V: U14.2 (S)
- no-connect marks 2 -> 5
Other:
- moved on the sheet: C26, C41, PS1

Commit message: Electronic
Rework: Fan, ESP32 Pinout, 15V Power,
Added: GPIO ISO, ESD
Parts:
- removed R40, R41: R, symbol Device:R
- removed R49: 33k, symbol Device:R
- removed R50: 66k, symbol Device:R
- removed U14: DMP3098L-7, footprint:SOT-23_L2.9-W1.3-P1.90-LS2.4-BR, symbol DMP3098L-7:DMP3098L-7
- added D7: D, symbol Device:D
- R48: value R -> 165
Connections:
- net +5V: now also D7.2 (A)
- net GND: now also U5.1 (GND); no longer J4.2 (Pin_2), PS1.2 (AC/N), U4.3 (~Neutral)
- net U: now also U10.3 (IP-)
- net VS: now also D7.1 (K)
- net W: now also U11.3 (IP-)
- net at U10.1 (IP+), U13.22 (U): now also U10.2 (IP+)
- net at K2.14, R1.2, U9.1 (IP+): now also U9.2 (IP+)
- net at U9.3 (IP-): now also U4.2 (~Phase), U9.4 (IP-)
- net at U11.1 (IP+), U13.20 (W): now also U11.2 (IP+)
- new net AC_N: J4.2 (Pin_2), PS1.2 (AC/N), U4.3 (~Neutral)
- no-connect marks 5 -> 7
Other:
- moved on the sheet: C21, C22, C24, C25, C39, C40, C41, D1, D2, D6, J4, L1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

Commit message: Electronic
Power Terminal edit
Parts:
- removed J4: Screw_Terminal_01x08, Connector_Phoenix_MC_HighVoltage:PhoenixContact_MCV_1,5_8-G-5.08_1x08_P5.08mm_Vertical, symbol Connector:Screw_Terminal_01x08
- added C51: C, symbol Device:C
- added H1, H2, H3, H4, H5, H6: MountingHole_Pad, MountingHole:MountingHole_3.2mm_M3_DIN965_Pad_TopBottom, symbol Mechanical:MountingHole_Pad
- added J10, J4: Screw_Terminal_01x04, Connector_Phoenix_MC_HighVoltage:PhoenixContact_MCV_1,5_4-G-5.08_1x04_P5.08mm_Vertical, symbol Connector:Screw_Terminal_01x04
- added J8, J9: Conn_01x01, Connector_PinHeader_2.54mm:PinHeader_1x01_P2.54mm_Vertical, symbol Connector_Generic:Conn_01x01
- added R40, R41: 10k, symbol Device:R
- added R60: 999m, symbol Device:R
- C1: footprint footprints:ESMQ351VSN102MA50S -> (none)
- C20: value C_Polarized -> C_P
- D1, D2: footprint (none) -> LED_SMD:LED_0603_1608Metric
- R10, R5, R6, R7, R8, R9: value R -> 165
- U4: footprint (none) -> Own_Library:LVE2560E
Connections:
- net +3.3V: now also R40.1, R41.1
- net AC_L: now also J10.1 (Pin_1)
- net AC_N: now also J10.2 (Pin_2)
- net Earth: now also H1.1, H2.1, H3.1, H4.1, H5.1, H6.1, J10.3 (Pin_3), J10.4 (Pin_4)
- net GND: now also C51.2, J4.1 (Pin_1), R60.2
- net U: now also J4.4 (Pin_4)
- net V: now also J4.3 (Pin_3)
- net VS: now also J9.1 (Pin_1)
- net W: now also J4.2 (Pin_2)
- net at C1.1, C2.1, C3.1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: now also J8.1 (Pin_1)
- net VFO: now reaches U13.14 (VFO)
- net VFO: now also R40.2
- net ITRIP: now reaches U13.15 (ITRIP)
- net ITRIP: now also C51.1, R41.2, R60.1
- no-connect marks 7 -> 8
Other:
- moved on the sheet: C20, C42, C43, C44, C45, C6, R44, R45, U10, U11

Commit message: Electronic
Footprint assignment
Parts:
- removed C20: C_P, symbol Device:C_Polarized
- added C20: 10uF, Capacitor_SMD:C_0201_0603Metric, symbol Device:C
- added C52: 1uF, Capacitor_SMD:C_0603_1608Metric, symbol Device:C
- added R61: 3.3k, Resistor_SMD:R_0201_0603Metric_Pad0.64x0.40mm_HandSolder, symbol Device:R
- added R62: 10k, Resistor_SMD:R_0201_0603Metric_Pad0.64x0.40mm_HandSolder, symbol Device:R
- C1: footprint (none) -> footprints:ESMQ351VSN102MA50S
- C10, C11, C12, C13, C8, C9: value C -> 10nF; footprint (none) -> Capacitor_SMD:C_0201_0603Metric
- C14, C17, C18: value C_Polarized -> 260uF
- C15, C16, C19: value C -> 100nF
- C21, C24, C51: value C -> 100nF; footprint (none) -> Capacitor_SMD:C_0603_1608Metric
- C22: value C -> 10uF; footprint (none) -> Capacitor_SMD:C_0603_1608Metric
- C25, C40: value C -> 22uF; footprint (none) -> Capacitor_SMD:C_0603_1608Metric
- C26, C41, C42, C43, C44, C45: footprint (none) -> Capacitor_SMD:C_0603_1608Metric
- C38, C39: value C -> 220nF; footprint (none) -> Capacitor_SMD:C_0603_1608Metric
- C6: value C -> 100nF; footprint (none) -> Capacitor_SMD:C_0201_0603Metric
- D4, D6, D7: footprint (none) -> Diode_SMD:D_SOD-123
- H1, H2, H3, H4, H5, H6: value MountingHole_Pad -> ~
- J10: value Screw_Terminal_01x04 -> Net; footprint Connector_Phoenix_MC_HighVoltage:PhoenixContact_MCV_1,5_4-G-5.08_1x04_P5.08mm_Vertical -> TerminalBlock_Phoenix:TerminalBlock_Phoenix_PT-1,5-4-5.0-H_1x04_P5.00mm_Horizontal
- J4: value Screw_Terminal_01x04 -> Motor; footprint Connector_Phoenix_MC_HighVoltage:PhoenixContact_MCV_1,5_4-G-5.08_1x04_P5.08mm_Vertical -> TerminalBlock_Phoenix:TerminalBlock_Phoenix_PT-1,5-4-5.0-H_1x04_P5.00mm_Horizontal
- J8: value Conn_01x01 -> U_ZK
- J9: value Conn_01x01 -> U_VS
- L1: value L -> 2.2uH; footprint (none) -> Inductor_SMD:L_Bourns_SRP7028A_7.3x6.6mm
- R10, R13, R14, R28, R5, R6, R7, R8, R9: footprint (none) -> Resistor_SMD:R_0201_0603Metric
- R11: value R -> 33.2k; footprint (none) -> Resistor_SMD:R_0201_0603Metric
- R12: value R -> 10k; footprint (none) -> Resistor_SMD:R_0201_0603Metric
- R18: footprint (none) -> Resistor_SMD:R_1206_3216Metric
- R33: value R -> 1.8k; footprint (none) -> Resistor_SMD:R_0201_0603Metric_Pad0.64x0.40mm_HandSolder
- R34: value R -> 10k; footprint (none) -> Resistor_SMD:R_0201_0603Metric_Pad0.64x0.40mm_HandSolder
- R35, R39, R40, R41, R43, R44, R45, R48, R60: footprint (none) -> Resistor_SMD:R_0201_0603Metric_Pad0.64x0.40mm_HandSolder
- R46: value R -> 100k; footprint (none) -> Resistor_SMD:R_0201_0603Metric_Pad0.64x0.40mm_HandSolder
- R47: value R -> 820; footprint (none) -> Resistor_SMD:R_0201_0603Metric_Pad0.64x0.40mm_HandSolder
Connections:
- net +15V: now also C20.1
- net +3.3V: now also R61.1; no longer U8.16 (AIN1/GPIO1)
- net GND: now also C20.2, C52.2, R62.2
- net at R35.1, U8.8 (DECAP): now also C52.1
- new net: R61.2, R62.1, U8.16 (AIN1/GPIO1)
Other:
- moved on the sheet: C1, C10, C11, C12, C13, C2, C22, C3, C39, C4, C51, C6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

Commit message: Electronic
Voltage messurment updated
Parts:
- added C53, C54, C55: C, symbol Device:C
- added R63, R64: 33k, Resistor_SMD:R_1206_3216Metric, symbol Device:R
- R41: value 10k -> 4,7k
- R46: value 100k -> 33k; footprint Resistor_SMD:R_0201_0603Metric_Pad0.64x0.40mm_HandSolder -> Resistor_SMD:R_1206_3216Metric
- R60: value 999m -> 330; footprint Resistor_SMD:R_0201_0603Metric_Pad0.64x0.40mm_HandSolder -> (none)
Connections:
- net GND: now also C53.2, C54.2, C55.2; no longer R60.2
- net ITRIP: no longer C51.1, R41.2, U13.15 (ITRIP)
- net at R47.1, U8.1 (AIN2/GPIO2): now also C55.1, R64.2; no longer R46.2
- net at R33.1, R34.2, U8.15 (AIN0/GPIO0): now also C54.1
- net at R61.2, R62.1, U8.16 (AIN1/GPIO1): now also C53.1
- net at U9.1 (IP+), U9.2 (IP+): now also U4.1 (VDD); no longer K2.14, R1.2
- net at U9.3 (IP-), U9.4 (IP-): now also C1.1, C2.1, C3.1, C4.1, J8.1 (Pin_1), U13.23 (P), R63.1; no longer U4.2 (~Phase)
- new net: K2.14, R1.2, U4.2 (~Phase)
- new net: R46.1, R63.2
- new net: R46.2, R64.1
- new net: C51.1, R41.2, R60.2, U13.15 (ITRIP)
Other:
- moved on the sheet: C1, C10, C11, C12, C13, C14, C15, C16, C17, C18, C19, C2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

Commit message: Electronic
docu
Parts:
- removed C1, C2, C3, C4: 1mF, footprints:ESMQ351VSN102MA50S, symbol Device:C
- added C1, C2, C3, C4: 1mF, Own_Footprint:ESMQ351VSN102MA50S, symbol Device:C_Polarized
Connections:
- net GND: now also C1.2, C2.2, C3.2, C4.2
- net at J8.1 (Pin_1), R63.1, U13.23 (P)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: now also C1.1, C2.1, C3.1, C4.1
Changed lines of the file:
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@@
     (stroke (width 0) (type default))
   )
-  (wire (pts (xy 222.25 127) (xy 222.25 196.85))
+  (wire (pts (xy 222.25 142.24) (xy 222.25 196.85))
     (stroke (width 0) (type default))
   )
@@
     (stroke (width 0) (type default))
   )
-  (wire (pts (xy 232.41 127) (xy 232.41 196.85))
+  (wire (pts (xy 232.41 134.62) (xy 232.41 196.85))
     (stroke (width 0) (type default))
   )
@@
     (stroke (width 0) (type default))
   )
-  (wire (pts (xy 212.09 106.68) (xy 212.09 119.38))
+  (wire (pts (xy 212.09 106.68) (xy 212.09 140.97))
     (stroke (width 0) (type default))
   )
@@
     (stroke (width 0) (type default))
   )
-  (wire (pts (xy 222.25 106.68) (xy 222.25 119.38))
+  (wire (pts (xy 222.25 106.68) (xy 222.25 134.62))
     (stroke (width 0) (type default))
   )
@@
     (stroke (width 0) (type default))
   )
-  (wire (pts (xy 232.41 106.68) (xy 232.41 119.38))
+  (wire (pts (xy 232.41 106.68) (xy 232.41 127))
     (stroke (width 0) (type default))
   )
@@
     (stroke (width 0) (type default))
   )
-  (wire (pts (xy 212.09 127) (xy 212.09 196.85))
+  (wire (pts (xy 212.09 148.59) (xy 212.09 196.85))
     (stroke (width 0) (type default))
   )
@@
     )
   )
-  (symbol (lib_id "Device:C") (at 222.25 123.19 0) (unit 1)
-    (in_bom yes) (on_board yes) (dnp no) (fields_autoplaced)
-    (property "Reference" "C2" (at 226.06 121.92 0)
-      (effects (font (size 1.27 1.27)) (justify left))
-    )
-    (property "Value" "1mF" (at 226.06 124.46 0)
-      (effects (font (size 1.27 1.27)) (justify left))
-    )
-    (property "Footprint" "footprints:ESMQ351VSN102MA50S" (at 223.2152 127 0)
-      (effects (font (size 1.27 1.27)) hide)
-    )
-    (property "Datasheet" "~" (at 222.25 123.19 0)
-      (effects (font (size 1.27 1.27)) hide)
-    )
-    (pin "1")
-    (pin "2")
-    (instances
-      (project "MecProInverter"
-        (path "/c9071429-8b0d-45bf-aa6d-71cc2b7f068c/c32f479b-361e-4c54-ac43-ed36ba4d4493"
-          (reference "C2") (unit 1)
-        )
-      )
-    )
-  )
   (symbol (lib_id "Device:R") (at 179.07 288.29 180) (unit 1)
     (in_bom yes) (on_board yes) (dnp no)
@@
     )
   )
+  (symbol (lib_id "Device:C_Polarized") (at 242.57 123.19 0) (unit 1)
+    (in_bom yes) (on_board yes) (dnp no) (fields_autoplaced)
+    (property "Reference" "C4" (at 246.38 121.031 0)
+      (effects (font (size 1.27 1.27)) (justify left))
+    )
+    (property "Value" "1mF" (at 246.38 123.571 0)
+      (effects (font (size 1.27 1.27)) (justify left))
+    )
+    (property "Footprint" "Own_Footprint:ESMQ351VSN102MA50S" (at 243.5352 127 0)
+      (effects (font (size 1.27 1.27)) hide)
+    )
+    (property "Datasheet" "~" (at 242.57 123.19 0)
+      (effects (font (size 1.27 1.27)) hide)
+    )
+    (pin "1")
+    (pin "2")
+    (instances
+      (project "MecProInverter"
+        (path "/c9071429-8b0d-45bf-aa6d-71cc2b7f068c/c32f479b-361e-4c54-ac43-ed36ba4d4493"
+          (reference "C4") (unit 1)
+        )
+      )
+    )
+  )
   (symbol (lib_id "Device:R") (at 62.23 134.62 90) (unit 1)
     (in_bom yes) (on_board yes) (dnp no)
@@
     )
   )
+  (symbol (lib_id "Device:C_Polarized") (at 222.25 138.43 0) (unit 1)
+    (in_bom yes) (on_board yes) (dnp no) (fields_autoplaced)
+    (property "Reference" "C2" (at 226.06 136.271 0)
+      (effects (font (size 1.27 1.27)) (justify left))
+    )
+    (property "Value" "1mF" (at 226.06 138.811 0)
+      (effects (font (size 1.27 1.27)) (justify left))
+    )
+    (property "Footprint" "Own_Footprint:ESMQ351VSN102MA50S" (at 223.2152 142.24 0)
+      (effects (font (size 1.27 1.27)) hide)
+    )
+    (property "Datasheet" "~" (at 222.25 138.43 0)
+      (effects (font (size 1.27 1.27)) hide)
+    )
+    (pin "1")
+    (pin "2")
+    (instances
+      (project "MecProInverter"
+        (path "/c9071429-8b0d-45bf-aa6d-71cc2b7f068c/c32f479b-361e-4c54-ac43-ed36ba4d4493"
+          (reference "C2") (unit 1)
+        )
+      )
+    )
+  )
   (symbol (lib_id "IKCM20L60GA:IKCM20L60GA") (at 358.14 143.51 0) (unit 1)
     (in_bom yes) (on_board yes) (dnp no) (fields_autoplaced)
@@
     )
   )
-  (symbol (lib_id "Device:C") (at 232.41 123.19 0) (unit 1)
-    (in_bom yes) (on_board yes) (dnp no) (fields_autoplaced)
-    (property "Reference" "C3" (at 236.22 121.92 0)
-      (effects (font (size 1.27 1.27)) (justify left))
-    )
-    (property "Value" "1mF" (at 236.22 124.46 0)
-      (effects (font (size 1.27 1.27)) (justify left))
-    )
-    (property "Footprint" "footprints:ESMQ351VSN102MA50S" (at 233.3752 127 0)
-      (effects (font (size 1.27 1.27)) hide)
-    )
-    (property "Datasheet" "~" (at 232.41 123.19 0)
-      (effects (font (size 1.27 1.27)) hide)
-    )
-    (pin "1")
-    (pin "2")
-    (instances
-      (project "MecProInverter"
-        (path "/c9071429-8b0d-45bf-aa6d-71cc2b7f068c/c32f479b-361e-4c54-ac43-ed36ba4d4493"
-          (reference "C3") (unit 1)
-        )
-      )
-    )
-  )
   (symbol (lib_id "Device:R") (at 264.16 156.21 270) (unit 1)
     (in_bom yes) (on_board yes) (dnp no)
@@
     )
   )
+  (symbol (lib_id "Device:C_Polarized") (at 232.41 130.81 0) (unit 1)
+    (in_bom yes) (on_board yes) (dnp no) (fields_autoplaced)
+    (property "Reference" "C3" (at 236.22 128.651 0)
+      (effects (font (size 1.27 1.27)) (justify left))
+    )
+    (property "Value" "1mF" (at 236.22 131.191 0)
+      (effects (font (size 1.27 1.27)) (justify left))
+    )
+    (property "Footprint" "Own_Footprint:ESMQ351VSN102MA50S" (at 233.3752 134.62 0)
+      (effects (font (size 1.27 1.27)) hide)
+    )
+    (property "Datasheet" "~" (at 232.41 130.81 0)
+      (effects (font (size 1.27 1.27)) hide)
+    )
+    (pin "1")
+    (pin "2")
+    (instances
+      (project "MecProInverter"
+        (path "/c9071429-8b0d-45bf-aa6d-71cc2b7f068c/c32f479b-361e-4c54-ac43-ed36ba4d4493"
+          (reference "C3") (unit 1)
+        )
+      )
+    )
+  )
   (symbol (lib_id "power:+3.3V") (at 571.5 144.78 270) (unit 1)
     (in_bom yes) (on_board yes) (dnp no) (fields_autoplaced)
@@
     )
   )
-  (symbol (lib_id "Device:C") (at 212.09 123.19 0) (unit 1)
-    (in_bom yes) (on_board yes) (dnp no) (fields_autoplaced)
-    (property "Reference" "C1" (at 215.9 121.92 0)
-      (effects (font (size 1.27 1.27)) (justify left))
-    )
-    (property "Value" "1mF" (at 215.9 124.46 0)
-      (effects (font (size 1.27 1.27)) (justify left))
-    )
-    (property "Footprint" "footprints:ESMQ351VSN102MA50S" (at 213.0552 127 0)
-      (effects (font (size 1.27 1.27)) hide)
-    )
-    (property "Datasheet" "~" (at 212.09 123.19 0)
-      (effects (font (size 1.27 1.27)) hide)
-    )
-    (pin "1")
-    (pin "2")
-    (instances
-      (project "MecProInverter"
-        (path "/c9071429-8b0d-45bf-aa6d-71cc2b7f068c/c32f479b-361e-4c54-ac43-ed36ba4d4493"
-          (reference "C1") (unit 1)
-        )
-      )
-    )
-  )
   (symbol (lib_id "Device:C") (at 189.23 119.38 180) (unit 1)
     (in_bom yes) (on_board yes) (dnp no)
@@
     )
   )
+  (symbol (lib_id "Device:C_Polarized") (at 212.09 144.78 0) (unit 1)
+    (in_bom yes) (on_board yes) (dnp no) (fields_autoplaced)
+    (property "Reference" "C1" (at 215.9 142.621 0)
+      (effects (font (size 1.27 1.27)) (justify left))
+    )
+    (property "Value" "1mF" (at 215.9 145.161 0)
+      (effects (font (size 1.27 1.27)) (justify left))
+    )
+    (property "Footprint" "Own_Footprint:ESMQ351VSN102MA50S" (at 213.0552 148.59 0)
+      (effects (font (size 1.27 1.27)) hide)
+    )
+    (property "Datasheet" "~" (at 212.09 144.78 0)
+      (effects (font (size 1.27 1.27)) hide)
+    )
+    (pin "1")
+    (pin "2")
+    (instances
+      (project "MecProInverter"
+        (path "/c9071429-8b0d-45bf-aa6d-71cc2b7f068c/c32f479b-361e-4c54-ac43-ed36ba4d4493"
+          (reference "C1") (unit 1)
+        )
+      )
+    )
+  )
   (symbol (lib_id "Device:C_Polarized") (at 316.23 118.11 270) (unit 1)
     (in_bom yes) (on_board yes) (dnp no) (fields_autoplaced)
@@
         )
       )
-    )
-  )
-  (symbol (lib_id "Device:C") (at 242.57 123.19 0) (unit 1)
-    (in_bom yes) (on_board yes) (dnp no) (fields_autoplaced)
-    (property "Reference" "C4" (at 246.38 121.92 0)
-      (effects (font (size 1.27 1.27)) (justify left))
-    )
-    (property "Value" "1mF" (at 246.38 124.46 0)
-      (effects (font (size 1.27 1.27)) (justify left))
-    )
-    (property "Footprint" "footprints:ESMQ351VSN102MA50S" (at 243.5352 127 0)
-      (effects (font (size 1.27 1.27)) hide)
-    )
-    (property "Datasheet" "~" (at 242.57 123.19 0)
-      (effects (font (size 1.27 1.27)) hide)
-    )
-    (pin "1")
-    (pin "2")
-    (instances
-      (project "MecProInverter"
-        (path "/c9071429-8b0d-45bf-aa6d-71cc2b7f068c/c32f479b-361e-4c54-ac43-ed36ba4d4493"
-          (reference "C4") (unit 1)
-        )
-      )

Commit message: Electronic
Added 3d Moodel on Layout
Parts:
- U4: footprint Own_Library:LVE2560E -> Own_Footprint:LVE2560E
Changed lines of the file:
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@@
       (effects (font (size 1.27 1.27)))
     )
-    (property "Footprint" "Own_Library:LVE2560E" (at 80.01 149.86 0)
+    (property "Footprint" "Own_Footprint:LVE2560E" (at 80.01 149.86 0)
       (effects (font (size 1.27 1.27)) hide)
     )
