File: electronic/MecProInverter/power.kicad_sch (KiCad schematic)
At the start: 92 parts, among them J10 Net, J4 Motor, J8 U_ZK, J9 U_VS, K2 RT314A12, Q1 DMN3404L, U10 CC6904SO-30A, U11 CC6904SO-30A, U13 IKCM20L60GA, U4 LVE2560E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

Commit message: Electronic
Schematic V1.0
Parts:
- removed C44: 0.1nF, Capacitor_SMD:C_0603_1608Metric, symbol Device:C
- added C56: 100nF, Capacitor_SMD:C_0603_1608Metric, symbol Device:C
- added D10, D11, D8, D9: D, Diode_SMD:D_0603_1608Metric, symbol Device:D
- added R65: 10M, Resistor_SMD:R_0603_1608Metric, symbol Device:R
- C10, C11, C12, C13, C20, C6, C8, C9: footprint Capacitor_SMD:C_0201_0603Metric -> Capacitor_SMD:C_0603_1608Metric
- C14, C17, C18: value 260uF -> 4.7uF; footprint (none) -> Capacitor_SMD:C_0603_1608Metric
- C15, C16, C19: footprint (none) -> Capacitor_SMD:C_0603_1608Metric
- C41, C42: value 0.1nF -> 100nF
- C53, C54, C55: value C -> 100nF; footprint (none) -> Capacitor_SMD:C_0603_1608Metric
- R1: footprint (none) -> Own_Footprint:PWR220T-20
- R10, R11, R12, R13, R14, R28, R5, R6, R7, R8, R9: footprint Resistor_SMD:R_0201_0603Metric -> Resistor_SMD:R_0603_1608Metric
- R33, R34, R39, R40, R41, R47, R48, R61, R62: footprint Resistor_SMD:R_0201_0603Metric_Pad0.64x0.40mm_HandSolder -> Resistor_SMD:R_0603_1608Metric
- R35: value 999m -> 999M; footprint Resistor_SMD:R_0201_0603Metric_Pad0.64x0.40mm_HandSolder -> Resistor_SMD:R_0603_1608Metric
- R43, R44, R45: value 100 -> 10M; footprint Resistor_SMD:R_0201_0603Metric_Pad0.64x0.40mm_HandSolder -> Resistor_SMD:R_0603_1608Metric
- R60: footprint (none) -> Resistor_SMD:R_0603_1608Metric
Connections:
- net AC_L: now also K2.14; no longer K2.11
- net CURRENT_AC: now also C56.2, D8.1 (K), R65.1; no longer C41.2, R43.2
- net GND: now also R43.2, R44.2, R45.2, C56.1, R65.2
- net at C55.1, U8.1 (AIN2/GPIO2): now also R45.1, D11.1 (K); no longer R47.1, R64.2
- net at U8.3 (AIN4/GPIO4): now also C42.2, R44.1, D10.1 (K); no longer R45.2
- net at U10.7 (OUT): now also D9.2 (A); no longer R44.1
- net at R43.1: now also C41.2, U8.2 (AIN3/GPIO3), D9.1 (K); no longer U9.7 (OUT)
- net at U11.7 (OUT): now also D10.2 (A); no longer R45.1
- net at R1.2, U4.2 (~Phase): now also K2.11; no longer K2.14
- new net: D8.2 (A), U9.7 (OUT)
- new net: D11.2 (A), R47.1, R64.2
Other:
- moved on the sheet: C20, C43, C51, C53, C55, C6, D4, H1, H2, H3, H4, H5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

Commit message: Electronic
PCB buy!!!
Parts:
- C1, C2, C4, H1, H2, H3, H4, H5, H6, J10, J4, J8, J9, K2, PS1, R1, U13, U4: now left out of the parts list
- C20, C22: value 10uF -> 22uF
- C38, C39: value 220nF -> 100nF
- R10, R48, R5, R6, R7, R8, R9: value 165 -> 121
- R11: value 33.2k -> 33k
- R13: value 40 -> 121
- R28: value 100k -> 10k
- R41: value 4,7k -> 3,3k
- R60: value 330 -> 121
Changed lines of the file:
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@@
       (effects (font (size 1.27 1.27)) (justify left))
     )
-    (property "Value" "100k" (at 26.67 118.11 90)
+    (property "Value" "10k" (at 26.67 118.11 90)
       (effects (font (size 1.27 1.27)) (justify left))
     )
@@
   )
   (symbol (lib_id "Connector_Generic:Conn_01x01") (at 443.23 294.64 90) (unit 1)
-    (in_bom yes) (on_board yes) (dnp no) (fields_autoplaced)
+    (in_bom no) (on_board yes) (dnp no) (fields_autoplaced)
     (property "Reference" "J9" (at 445.77 293.37 90)
       (effects (font (size 1.27 1.27)) (justify right))
@@
   )
   (symbol (lib_id "Converter_ACDC:IRM-20-15") (at 387.35 302.26 0) (unit 1)
-    (in_bom yes) (on_board yes) (dnp no) (fields_autoplaced)
+    (in_bom no) (on_board yes) (dnp no) (fields_autoplaced)
     (property "Reference" "PS1" (at 387.35 293.37 0)
       (effects (font (size 1.27 1.27)))
@@
   )
   (symbol (lib_id "Mechanical:MountingHole_Pad") (at 542.29 294.64 0) (unit 1)
-    (in_bom yes) (on_board yes) (dnp no) (fields_autoplaced)
+    (in_bom no) (on_board yes) (dnp no) (fields_autoplaced)
     (property "Reference" "H2" (at 544.83 293.37 0)
       (effects (font (size 1.27 1.27)) (justify left))
@@
       (effects (font (size 1.27 1.27)) (justify right))
     )
-    (property "Value" "220nF" (at 572.77 171.45 0)
+    (property "Value" "100nF" (at 572.77 171.45 0)
       (effects (font (size 1.27 1.27)) (justify right))
     )
@@
       (effects (font (size 1.27 1.27)))
     )
-    (property "Value" "165" (at 26.67 95.25 90)
+    (property "Value" "121" (at 26.67 95.25 90)
       (effects (font (size 1.27 1.27)))
     )
@@
   )
   (symbol (lib_id "Relay:RT314A12") (at 55.88 90.17 0) (unit 1)
-    (in_bom yes) (on_board yes) (dnp no) (fields_autoplaced)
+    (in_bom no) (on_board yes) (dnp no) (fields_autoplaced)
     (property "Reference" "K2" (at 40.64 90.17 90)
       (effects (font (size 1.27 1.27)))
@@
       (effects (font (size 1.27 1.27)))
     )
-    (property "Value" "33.2k" (at 184.15 289.56 0)
+    (property "Value" "33k" (at 184.15 289.56 0)
       (effects (font (size 1.27 1.27)))
     )
@@
   )
   (symbol (lib_id "LVE2560E:LVE2560E") (at 87.63 149.86 0) (unit 1)
-    (in_bom yes) (on_board yes) (dnp no)
+    (in_bom no) (on_board yes) (dnp no)
     (property "Reference" "U4" (at 99.06 119.38 0)
       (effects (font (size 1.27 1.27)))
@@
   )
   (symbol (lib_id "Mechanical:MountingHole_Pad") (at 542.29 308.61 180) (unit 1)
-    (in_bom yes) (on_board yes) (dnp no) (fields_autoplaced)
+    (in_bom no) (on_board yes) (dnp no) (fields_autoplaced)
     (property "Reference" "H5" (at 544.83 309.88 0)
       (effects (font (size 1.27 1.27)) (justify right))
@@
   )
   (symbol (lib_id "Mechanical:MountingHole_Pad") (at 565.15 294.64 0) (unit 1)
-    (in_bom yes) (on_board yes) (dnp no) (fields_autoplaced)
+    (in_bom no) (on_board yes) (dnp no) (fields_autoplaced)
     (property "Reference" "H3" (at 567.69 293.37 0)
       (effects (font (size 1.27 1.27)) (justify left))
@@
       (effects (font (size 1.27 1.27)))
     )
-    (property "Value" "165" (at 271.78 153.67 90)
+    (property "Value" "121" (at 271.78 153.67 90)
       (effects (font (size 1.27 1.27)))
     )
@@
     )
     (property "Value" "100nF" (at 406.4 168.91 0)
-      (effects (font (size 1.27 1.27)) (justify left) hide)
+      (effects (font (size 1.27 1.27)) (justify left))
     )
     (property "Footprint" "Capacitor_SMD:C_0603_1608Metric" (at 404.8252 171.45 0)
@@
   )
   (symbol (lib_id "Connector:Screw_Terminal_01x04") (at 246.38 303.53 180) (unit 1)
-    (in_bom yes) (on_board yes) (dnp no)
+    (in_bom no) (on_board yes) (dnp no)
     (property "Reference" "J10" (at 246.38 293.37 0)
       (effects (font (size 1.27 1.27)))
@@
       (effects (font (size 1.27 1.27)))
     )
-    (property "Value" "165" (at 271.78 146.05 90)
+    (property "Value" "121" (at 271.78 146.05 90)
       (effects (font (size 1.27 1.27)))
     )
@@
   )
   (symbol (lib_id "Mechanical:MountingHole_Pad") (at 519.43 307.34 180) (unit 1)
-    (in_bom yes) (on_board yes) (dnp no) (fields_autoplaced)
+    (in_bom no) (on_board yes) (dnp no) (fields_autoplaced)
     (property "Reference" "H4" (at 521.97 308.61 0)
       (effects (font (size 1.27 1.27)) (justify right))
@@
   )
   (symbol (lib_id "Device:C_Polarized") (at 242.57 123.19 0) (unit 1)
-    (in_bom yes) (on_board yes) (dnp no) (fields_autoplaced)
+    (in_bom no) (on_board yes) (dnp no) (fields_autoplaced)
     (property "Reference" "C4" (at 246.38 121.031 0)
       (effects (font (size 1.27 1.27)) (justify left))
@@
   )
   (symbol (lib_id "Device:R") (at 69.85 134.62 90) (unit 1)
-    (in_bom yes) (on_board yes) (dnp no)
+    (in_bom no) (on_board yes) (dnp no)
     (property "Reference" "R1" (at 69.85 132.08 90)
       (effects (font (size 1.27 1.27)))
@@
       (effects (font (size 1.27 1.27)) (justify left))
     )
-    (property "Value" "10uF" (at 113.03 303.53 0)
+    (property "Value" "22uF" (at 113.03 303.53 0)
       (effects (font (size 1.27 1.27)) (justify left))
     )
@@
   )
   (symbol (lib_id "Device:C_Polarized") (at 222.25 138.43 0) (unit 1)
-    (in_bom yes) (on_board yes) (dnp no) (fields_autoplaced)
+    (in_bom no) (on_board yes) (dnp no) (fields_autoplaced)
     (property "Reference" "C2" (at 226.06 136.271 0)
       (effects (font (size 1.27 1.27)) (justify left))
@@
   )
   (symbol (lib_id "IKCM20L60GA:IKCM20L60GA") (at 358.14 143.51 0) (unit 1)
-    (in_bom yes) (on_board yes) (dnp no) (fields_autoplaced)
+    (in_bom no) (on_board yes) (dnp no) (fields_autoplaced)
     (property "Reference" "U13" (at 356.87 120.65 0)
       (effects (font (size 1.27 1.27)))
@@
       (effects (font (size 1.27 1.27)))
     )
-    (property "Value" "165" (at 279.4 151.13 90)
+    (property "Value" "121" (at 279.4 151.13 90)
       (effects (font (size 1.27 1.27)))
     )
@@
       (effects (font (size 1.27 1.27)) (justify left))
     )
-    (property "Value" "330" (at 383.54 147.32 0)
+    (property "Value" "121" (at 383.54 147.32 0)
       (effects (font (size 1.27 1.27)) (justify left))
     )
@@
       (effects (font (size 1.27 1.27)))
     )
-    (property "Value" "165" (at 264.16 156.21 90)
+    (property "Value" "121" (at 264.16 156.21 90)
       (effects (font (size 1.27 1.27)))
     )
@@
   )
   (symbol (lib_id "Connector:Screw_Terminal_01x04") (at 246.38 285.75 180) (unit 1)
-    (in_bom yes) (on_board yes) (dnp no) (fields_autoplaced)
+    (in_bom no) (on_board yes) (dnp no) (fields_autoplaced)
     (property "Reference" "J4" (at 246.38 274.32 0)
       (effects (font (size 1.27 1.27)))
@@
       (effects (font (size 1.27 1.27)) (justify left))
     )
-    (property "Value" "10uF" (at 393.7 179.07 0)
+    (property "Value" "22uF" (at 393.7 179.07 0)
       (effects (font (size 1.27 1.27)) (justify left))
     )
@@
       (effects (font (size 1.27 1.27)))
     )
-    (property "Value" "165" (at 264.16 148.59 90)
+    (property "Value" "121" (at 264.16 148.59 90)
       (effects (font (size 1.27 1.27)))
     )
@@
       (effects (font (size 1.27 1.27)) (justify left))
     )
-    (property "Value" "4,7k" (at 406.4 147.32 0)
+    (property "Value" "3,3k" (at 406.4 147.32 0)
       (effects (font (size 1.27 1.27)) (justify left))
     )
@@
       (effects (font (size 1.27 1.27)) (justify left))
     )
-    (property "Value" "40" (at 307.34 294.64 0)
+    (property "Value" "121" (at 307.34 294.64 0)
       (effects (font (size 1.27 1.27)) (justify left))
     )
@@
   )
   (symbol (lib_id "Mechanical:MountingHole_Pad") (at 519.43 295.91 0) (unit 1)
-    (in_bom yes) (on_board yes) (dnp no)
+    (in_bom no) (on_board yes) (dnp no)
     (property "Reference" "H1" (at 521.97 292.1 0)
       (effects (font (size 1.27 1.27)) (justify left))
@@
   )
   (symbol (lib_id "Connector_Generic:Conn_01x01") (at 212.09 73.66 90) (unit 1)
-    (in_bom yes) (on_board yes) (dnp no) (fields_autoplaced)
+    (in_bom no) (on_board yes) (dnp no) (fields_autoplaced)
     (property "Reference" "J8" (at 214.63 72.39 90)
       (effects (font (size 1.27 1.27)) (justify right))
@@
       (effects (font (size 1.27 1.27)) hide)
     )
+    (property "Sim.Enable" "0" (at 232.41 130.81 0)
+      (effects (font (size 1.27 1.27)) hide)
+    )
     (pin "1")
     (pin "2")
@@
       (effects (font (size 1.27 1.27)))
     )
-    (property "Value" "165" (at 279.4 143.51 90)
+    (property "Value" "121" (at 279.4 143.51 90)
       (effects (font (size 1.27 1.27)))
     )
@@
   )
   (symbol (lib_id "Mechanical:MountingHole_Pad") (at 565.15 308.61 180) (unit 1)
-    (in_bom yes) (on_board yes) (dnp no) (fields_autoplaced)
+    (in_bom no) (on_board yes) (dnp no) (fields_autoplaced)
     (property "Reference" "H6" (at 567.69 309.88 0)
       (effects (font (size 1.27 1.27)) (justify right))
@@
   )
   (symbol (lib_id "Device:C_Polarized") (at 212.09 144.78 0) (unit 1)
-    (in_bom yes) (on_board yes) (dnp no) (fields_autoplaced)
+    (in_bom no) (on_board yes) (dnp no) (fields_autoplaced)
     (property "Reference" "C1" (at 215.9 142.621 0)
       (effects (font (size 1.27 1.27)) (justify left))
@@
       (effects (font (size 1.27 1.27)) (justify left))
     )
-    (property "Value" "220nF" (at 524.51 172.72 0)
+    (property "Value" "100nF" (at 524.51 172.72 0)
       (effects (font (size 1.27 1.27)) (justify left))
     )
