File: electronic/MecProInverter/control.kicad_sch (KiCad schematic)
At the start: 85 parts, among them J1 0022232031, J2 0022232031, J3 Screw_Terminal_01x06, J5 Conn_01x08, J6 LM61, J7 Conn_01x11, Q1 DMN3404L, SW1 PTS645SM95SMTR92LFS, SW2 PTS645SM95SMTR92LFS, SW3 PTS645SM95SMTR92LFS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

Commit message: Electronic
Power Terminal edit
Parts:
- added U19, U20: PSRV05-4MR6T1G, footprint:SOT-23-6_L2.9-W1.6-P0.95-LS2.8-BL, symbol PSRV05-4MR6T1G:PSRV05-4MR6T1G
- J1, J2: footprint digikey-footprints:PinHeader_1x3_P2.54mm_Drill1.02mm -> footprint:CONN-TH_3P-P2.54_22-23-2031
- J3: footprint (none) -> Connector_Phoenix_MC_HighVoltage:PhoenixContact_MCV_1,5_6-G-5.08_1x06_P5.08mm_Vertical
- RV1: footprint (none) -> Potentiometer_THT:Potentiometer_Alps_RK09K_Single_Vertical
- TP1, TP2, TP3, TP4, TP5, TP6, TP7, TP8: footprint Connector_Pin:Pin_D1.0mm_L10.0mm_LooseFit -> TestPoint:TestPoint_Pad_D2.0mm
Connections:
- net +3.3V: now also U19.5, U20.5
- net GND: now also U19.2, U20.2
- net I2C_SCL: now also U19.6
- net I2C_SDA: now also U19.4
- net SPI_CLK: now also U20.1
- net SPI_CS: now also U20.3
- net SPI_MISO: now also U20.4
- net SPI_MOSI: now also U20.6
- net UART_RX: now also U19.1
- net UART_TX: now also U19.3
- net VFO: now reaches U1.27 (IO47)
- net ITRIP: now reaches U1.28 (IO33)
- no-connect marks 8 -> 17
Other:
- moved on the sheet: J7, R2, R3

Commit message: Electronic
Footprint assignment
Parts:
- C23, C27, C28, C29, C30, C31, C33, C34, C35, C36, C46, C47, C48, C49, C50: footprint (none) -> Capacitor_SMD:C_0603_1608Metric
- C32: value C -> 1uF; footprint (none) -> Capacitor_SMD:C_0603_1608Metric
- C37: value 100uF -> 10uF; footprint (none) -> Capacitor_SMD:C_0603_1608Metric
- C5, C7: footprint (none) -> Capacitor_SMD:C_0201_0603Metric
- D5: footprint (none) -> Diode_SMD:D_SOD-123
- J3: value Screw_Terminal_01x06 -> ISO_Data; footprint Connector_Phoenix_MC_HighVoltage:PhoenixContact_MCV_1,5_6-G-5.08_1x06_P5.08mm_Vertical -> TerminalBlock_Phoenix:TerminalBlock_Phoenix_MPT-0,5-6-2.54_1x06_P2.54mm_Horizontal
- J5: value Conn_01x08 -> Display
- J6: value LM61 -> MAX312820
- J7: value Conn_01x11 -> Test
- R15, R16, R17, R19, R2, R20, R21, R22, R23, R24, R25, R26, R27, R29, R3, R30, R4: footprint (none) -> Resistor_SMD:R_0201_0603Metric
- R31: footprint (none) -> Resistor_SMD:R_1206_3216Metric
- R32, R36, R37, R38, R42, R49, R50, R51, R52, R57, R58, R59: footprint (none) -> Resistor_SMD:R_0201_0603Metric_Pad0.64x0.40mm_HandSolder
- R53, R54, R55, R56: value R -> 0; footprint (none) -> Resistor_SMD:R_0201_0603Metric_Pad0.64x0.40mm_HandSolder
- renumbered J2 to Fan1, J1 to Fan2

Commit message: Electronic
Voltage messurment updated
Parts:
- removed RV1: 10K, Potentiometer_THT:Potentiometer_Alps_RK09K_Single_Vertical, symbol Device:R_Potentiometer
- added U21: RK09D113000F_10k, footprint:RES-ADJ-TH_RK09D1130C4G, symbol RK09D113000F:RK09D113000F
Connections:
- net +3.3V: now also U21.1
- net FAN1_PWM_FB: now also U1.30 (IO48); no longer U1.6 (IO2)
- net FAN2_PWM_FB: now also U1.27 (IO47); no longer U1.7 (IO3)
- net GND: now also U21.3, U21.4, U21.5
- net POT1OUT: now also U21.2
- net VFO: now also U1.6 (IO2); no longer U1.27 (IO47)
- no-connect marks 17 -> 16
Changed lines of the file:
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@@
   (junction (at 391.16 308.61) (diameter 0) (color 0 0 0 0)
   )
+  (junction (at 90.17 374.65) (diameter 0) (color 0 0 0 0)
+  )
   (junction (at 255.27 360.68) (diameter 0) (color 0 0 0 0)
   )
@@
   (junction (at 104.14 113.03) (diameter 0) (color 0 0 0 0)
   )
+  (junction (at 67.31 374.65) (diameter 0) (color 0 0 0 0)
+  )
   (junction (at 59.69 130.81) (diameter 0) (color 0 0 0 0)
   )
@@
   (junction (at 518.16 69.85) (diameter 0) (color 0 0 0 0)
   )
-  (junction (at 90.17 374.65) (diameter 0) (color 0 0 0 0)
-  )
   (junction (at 90.17 349.25) (diameter 0) (color 0 0 0 0)
   )
@@
   (junction (at 528.32 120.65) (diameter 0) (color 0 0 0 0)
   )
+  (junction (at 67.31 372.11) (diameter 0) (color 0 0 0 0)
+  )
   (junction (at 525.78 67.31) (diameter 0) (color 0 0 0 0)
   )
   (no_connect (at 50.8 339.09))
   (no_connect (at 66.04 351.79))
-  (no_connect (at 196.85 133.35))
   (no_connect (at 471.17 105.41))
   (no_connect (at 196.85 125.73))
@@
     (stroke (width 0) (type default))
   )
+  (wire (pts (xy 195.58 133.35) (xy 185.42 133.35))
+    (stroke (width 0) (type default))
+  )
   (wire (pts (xy 53.34 232.41) (xy 119.38 232.41))
     (stroke (width 0) (type default))
@@
     (stroke (width 0) (type default))
   )
-  (wire (pts (xy 62.23 374.65) (xy 90.17 374.65))
-    (stroke (width 0) (type default))
-  )
   (wire (pts (xy 92.71 110.49) (xy 115.57 110.49))
     (stroke (width 0) (type default))
@@
     (stroke (width 0) (type default))
   )
+  (wire (pts (xy 63.5 372.11) (xy 67.31 372.11))
+    (stroke (width 0) (type default))
+  )
   (wire (pts (xy 185.42 115.57) (xy 196.85 115.57))
     (stroke (width 0) (type default))
@@
     (stroke (width 0) (type default))
   )
+  (wire (pts (xy 63.5 374.65) (xy 67.31 374.65))
+    (stroke (width 0) (type default))
+  )
   (wire (pts (xy 144.78 118.11) (xy 154.94 118.11))
     (stroke (width 0) (type default))
@@
     (stroke (width 0) (type default))
   )
+  (wire (pts (xy 195.58 130.81) (xy 185.42 130.81))
+    (stroke (width 0) (type default))
+  )
   (wire (pts (xy 88.9 222.25) (xy 88.9 186.69))
     (stroke (width 0) (type default))
@@
     (stroke (width 0) (type default))
   )
+  (wire (pts (xy 144.78 95.25) (xy 154.94 95.25))
+    (stroke (width 0) (type default))
+  )
   (wire (pts (xy 402.59 214.63) (xy 402.59 205.74))
     (stroke (width 0) (type default))
@@
     (stroke (width 0) (type default))
   )
+  (wire (pts (xy 90.17 367.03) (xy 90.17 374.65))
+    (stroke (width 0) (type default))
+  )
   (wire (pts (xy 518.16 64.77) (xy 533.4 64.77))
     (stroke (width 0) (type default))
@@
     (stroke (width 0) (type default))
   )
+  (wire (pts (xy 49.53 372.11) (xy 49.53 365.76))
+    (stroke (width 0) (type default))
+  )
   (wire (pts (xy 523.24 193.04) (xy 532.13 193.04))
     (stroke (width 0) (type default))
@@
     (stroke (width 0) (type default))
   )
+  (wire (pts (xy 58.42 379.73) (xy 58.42 384.81))
+    (stroke (width 0) (type default))
+  )
   (wire (pts (xy 193.04 312.42) (xy 220.98 312.42))
     (stroke (width 0) (type default))
@@
     (stroke (width 0) (type default))
   )
-  (wire (pts (xy 144.78 97.79) (xy 154.94 97.79))
-    (stroke (width 0) (type default))
-  )
   (wire (pts (xy 193.04 372.11) (xy 220.98 372.11))
     (stroke (width 0) (type default))
@@
     (stroke (width 0) (type default))
   )
-  (wire (pts (xy 185.42 130.81) (xy 210.82 130.81))
-    (stroke (width 0) (type default))
-  )
   (wire (pts (xy 224.79 322.58) (xy 252.73 322.58))
     (stroke (width 0) (type default))
@@
     (stroke (width 0) (type default))
   )
-  (wire (pts (xy 90.17 374.65) (xy 90.17 377.19))
-    (stroke (width 0) (type default))
-  )
   (wire (pts (xy 374.65 25.4) (xy 374.65 29.21))
     (stroke (width 0) (type default))
@@
     (stroke (width 0) (type default))
   )
-  (wire (pts (xy 58.42 378.46) (xy 58.42 384.81))
+  (wire (pts (xy 408.94 320.04) (xy 391.16 320.04))
     (stroke (width 0) (type default))
   )
-  (wire (pts (xy 408.94 320.04) (xy 391.16 320.04))
+  (wire (pts (xy 53.34 372.11) (xy 49.53 372.11))
     (stroke (width 0) (type default))
   )
@@
     (stroke (width 0) (type default))
   )
-  (wire (pts (xy 185.42 133.35) (xy 196.85 133.35))
-    (stroke (width 0) (type default))
-  )
   (wire (pts (xy 476.25 160.02) (xy 472.44 160.02))
     (stroke (width 0) (type default))
@@
     (stroke (width 0) (type default))
   )
-  (wire (pts (xy 472.44 172.72) (xy 472.44 179.07))
+  (wire (pts (xy 67.31 365.76) (xy 67.31 372.11))
     (stroke (width 0) (type default))
   )
-  (wire (pts (xy 144.78 130.81) (xy 154.94 130.81))
+  (wire (pts (xy 472.44 172.72) (xy 472.44 179.07))
     (stroke (width 0) (type default))
   )
-  (wire (pts (xy 54.61 374.65) (xy 44.45 374.65))
+  (wire (pts (xy 144.78 130.81) (xy 154.94 130.81))
     (stroke (width 0) (type default))
   )
@@
     (stroke (width 0) (type default))
   )
+  (wire (pts (xy 44.45 374.65) (xy 53.34 374.65))
+    (stroke (width 0) (type default))
+  )
   (wire (pts (xy 90.17 384.81) (xy 109.22 384.81))
     (stroke (width 0) (type default))
@@
     (stroke (width 0) (type default))
   )
-  (wire (pts (xy 90.17 374.65) (xy 90.17 367.03))
-    (stroke (width 0) (type default))
-  )
   (wire (pts (xy 53.34 245.11) (xy 73.66 245.11))
     (stroke (width 0) (type default))
@@
     (stroke (width 0) (type default))
   )
-  (wire (pts (xy 144.78 95.25) (xy 154.94 95.25))
-    (stroke (width 0) (type default))
-  )
   (wire (pts (xy 53.34 101.6) (xy 53.34 104.14))
     (stroke (width 0) (type default))
@@
     (stroke (width 0) (type default))
   )
+  (wire (pts (xy 90.17 374.65) (xy 90.17 377.19))
+    (stroke (width 0) (type default))
+  )
   (wire (pts (xy 83.82 349.25) (xy 90.17 349.25))
     (stroke (width 0) (type default))
@@
     (stroke (width 0) (type default))
   )
+  (wire (pts (xy 67.31 374.65) (xy 90.17 374.65))
+    (stroke (width 0) (type default))
+  )
   (wire (pts (xy 528.32 52.07) (xy 378.46 52.07))
     (stroke (width 0) (type default))
@@
     (stroke (width 0) (type default))
   )
+  (wire (pts (xy 67.31 372.11) (xy 67.31 374.65))
+    (stroke (width 0) (type default))
+  )
+  (wire (pts (xy 49.53 365.76) (xy 67.31 365.76))
+    (stroke (width 0) (type default))
+  )
   (wire (pts (xy 471.17 69.85) (xy 497.84 69.85))
     (stroke (width 0) (type default))
@@
     (effects (font (size 1.27 1.27)) (justify left bottom))
   )
-  (label "FAN2_PWM_FB" (at 144.78 97.79 180) (fields_autoplaced)
-    (effects (font (size 1.27 1.27)) (justify right bottom))
+  (label "FAN2_PWM_FB" (at 195.58 130.81 0) (fields_autoplaced)
+    (effects (font (size 1.27 1.27)) (justify left bottom))
   )
   (label "SW2OUT" (at 144.78 105.41 180) (fields_autoplaced)
@@
     (effects (font (size 1.27 1.27)) (justify left bottom))
   )
-  (label "FAN1_PWM_FB" (at 144.78 95.25 180) (fields_autoplaced)
-    (effects (font (size 1.27 1.27)) (justify right bottom))
+  (label "FAN1_PWM_FB" (at 195.58 133.35 0) (fields_autoplaced)
+    (effects (font (size 1.27 1.27)) (justify left bottom))
   )
   (label "SPI_CS" (at 73.66 240.03 0) (fields_autoplaced)
@@
     )
   )
-  (global_label "VFO" (shape input) (at 210.82 130.81 0) (fields_autoplaced)
-    (effects (font (size 1.27 1.27)) (justify left))
-    (property "Intersheetrefs" "${INTERSHEET_REFS}" (at 217.3129 130.81 0)
-      (effects (font (size 1.27 1.27)) (justify left) hide)
+  (global_label "VFO" (shape input) (at 144.78 95.25 180) (fields_autoplaced)
+    (effects (font (size 1.27 1.27)) (justify right))
+    (property "Intersheetrefs" "${INTERSHEET_REFS}" (at 138.2871 95.25 0)
+      (effects (font (size 1.27 1.27)) (justify right) hide)
     )
   )
@@
     )
   )
-  (symbol (lib_id "Device:R_Potentiometer") (at 58.42 374.65 270) (unit 1)
-    (in_bom yes) (on_board yes) (dnp no) (fields_autoplaced)
-    (property "Reference" "RV1" (at 58.42 368.3 90)
-      (effects (font (size 1.27 1.27)))
-    )
-    (property "Value" "10K" (at 58.42 370.84 90)
-      (effects (font (size 1.27 1.27)))
-    )
-    (property "Footprint" "Potentiometer_THT:Potentiometer_Alps_RK09K_Single_Vertical" (at 58.42 374.65 0)
-      (effects (font (size 1.27 1.27)) hide)
-    )
-    (property "Datasheet" "~" (at 58.42 374.65 0)
-      (effects (font (size 1.27 1.27)) hide)
-    )
-    (pin "1")
-    (pin "2")
-    (pin "3")
-    (instances
-      (project "MecProInverter"
-        (path "/c9071429-8b0d-45bf-aa6d-71cc2b7f068c/87c5d68c-a194-45d1-987f-2b491b6ac1ab"
-          (reference "RV1") (unit 1)
-        )
-      )
-    )
-  )
   (symbol (lib_id "power:+3.3V") (at 111.76 195.58 0) (unit 1)
     (in_bom yes) (on_board yes) (dnp no)
@@
         )
       )
+    )
+  )
+  (symbol (lib_id "RK09D113000F:RK09D113000F") (at 57.15 374.65 180) (unit 1)
+    (in_bom yes) (on_board yes) (dnp no) (fields_autoplaced)
+    (property "Reference" "U21" (at 58.166 367.03 0)
+      (effects (font (size 1.27 1.27)))
+    )
+    (property "Value" "RK09D113000F_10k" (at 58.166 369.57 0)
+      (effects (font (size 1.27 1.27)))
+    )
+    (property "Footprint" "footprint:RES-ADJ-TH_RK09D1130C4G" (at 57.15 364.49 0)
+      (effects (font (size 1.27 1.27) italic) hide)
+    )
+    (property "Datasheet" "https://atta.szlcsc.com/upload/public/pdf/source/20210222/C2687325_4FFD17AAA104A4955DD1E89BBAB92083.pdf" (at 59.436 374.777 0)
+      (effects (font (size 1.27 1.27)) (justify left) hide)
+    )
+    (property "LCSC" "C470317" (at 57.15 374.65 0)
+      (effects (font (size 1.27 1.27)) hide)
+    )
+    (pin "1")
+    (pin "2")
+    (pin "3")
+    (pin "4")
+    (pin "5")
+    (instances
+      (project "MecProInverter"
+        (path "/c9071429-8b0d-45bf-aa6d-71cc2b7f068c/87c5d68c-a194-45d1-987f-2b491b6ac1ab"
+          (reference "U21") (unit 1)
+        )
+      )

Commit message: Electronic
Added 3d Moodel on Layout
Parts:
- J5: footprint Connector_PinSocket_2.54mm:PinSocket_1x08_P2.54mm_Vertical -> Own_Footprint:Adafruit_938
Changed lines of the file:
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@@
       (effects (font (size 1.27 1.27)) (justify left))
     )
-    (property "Footprint" "Connector_PinSocket_2.54mm:PinSocket_1x08_P2.54mm_Vertical" (at 523.24 309.88 0)
+    (property "Footprint" "Own_Footprint:Adafruit_938" (at 523.24 309.88 0)
       (effects (font (size 1.27 1.27)) hide)
     )

Commit message: Electronic
Schematic V1.0
Parts:
- C5, C7: footprint Capacitor_SMD:C_0201_0603Metric -> Capacitor_SMD:C_0603_1608Metric
- R15, R16, R17, R19, R2, R20, R21, R22, R23, R24, R25, R26, R27, R29, R3, R30, R4: footprint Resistor_SMD:R_0201_0603Metric -> Resistor_SMD:R_0603_1608Metric
- R32, R36, R37, R38, R42, R49, R50, R51, R52, R53, R54, R55, R56, R57, R58, R59: footprint Resistor_SMD:R_0201_0603Metric_Pad0.64x0.40mm_HandSolder -> Resistor_SMD:R_0603_1608Metric
- TP1, TP2, TP3, TP4, TP5, TP6, TP7, TP8: footprint TestPoint:TestPoint_Pad_D2.0mm -> TestPoint:TestPoint_Pad_D1.5mm

Commit message: Electronic
Added USB-C CC Resistor
Parts:
- added R66, R67: 5.1k, Resistor_SMD:R_0603_1608Metric, symbol Device:R
Connections:
- net GNDD: now also R66.2, R67.2
- net at U3.10 (CC2): now also R66.1
- net at U3.4 (CC1): now also R67.1
- no-connect marks 16 -> 14
Changed lines of the file:
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@@
   (junction (at 434.34 161.29) (diameter 0) (color 0 0 0 0)
   )
+  (junction (at 496.57 120.65) (diameter 0) (color 0 0 0 0)
+  )
+  (junction (at 486.41 120.65) (diameter 0) (color 0 0 0 0)
+  )
   (junction (at 53.34 82.55) (diameter 0) (color 0 0 0 0)
   )
@@
   (no_connect (at 533.4 57.15))
   (no_connect (at 196.85 97.79))
-  (no_connect (at 533.4 59.69))
   (no_connect (at 66.04 316.23))
   (no_connect (at 50.8 356.87))
-  (no_connect (at 533.4 74.93))
   (no_connect (at 533.4 72.39))
   (no_connect (at 66.04 334.01))
@@
     (stroke (width 0) (type default))
   )
+  (wire (pts (xy 486.41 106.68) (xy 486.41 120.65))
+    (stroke (width 0) (type default))
+  )
   (wire (pts (xy 353.06 62.23) (xy 359.41 62.23))
     (stroke (width 0) (type default))
@@
     (stroke (width 0) (type default))
   )
+  (wire (pts (xy 496.57 74.93) (xy 496.57 99.06))
+    (stroke (width 0) (type default))
+  )
   (wire (pts (xy 515.62 72.39) (xy 525.78 72.39))
     (stroke (width 0) (type default))
@@
     (stroke (width 0) (type default))
   )
+  (wire (pts (xy 486.41 59.69) (xy 486.41 99.06))
+    (stroke (width 0) (type default))
+  )
   (wire (pts (xy 53.34 80.01) (xy 53.34 82.55))
     (stroke (width 0) (type default))
@@
     (stroke (width 0) (type default))
   )
+  (wire (pts (xy 533.4 74.93) (xy 496.57 74.93))
+    (stroke (width 0) (type default))
+  )
   (wire (pts (xy 561.34 41.91) (xy 528.32 41.91))
     (stroke (width 0) (type default))
@@
     (stroke (width 0) (type default))
   )
+  (wire (pts (xy 533.4 59.69) (xy 486.41 59.69))
+    (stroke (width 0) (type default))
+  )
   (wire (pts (xy 525.78 62.23) (xy 525.78 67.31))
     (stroke (width 0) (type default))
@@
     (stroke (width 0) (type default))
   )
-  (wire (pts (xy 463.55 120.65) (xy 516.89 120.65))
+  (wire (pts (xy 463.55 120.65) (xy 486.41 120.65))
     (stroke (width 0) (type default))
   )
@@
     (stroke (width 0) (type default))
   )
+  (wire (pts (xy 496.57 120.65) (xy 516.89 120.65))
+    (stroke (width 0) (type default))
+  )
   (wire (pts (xy 367.03 91.44) (xy 353.06 91.44))
     (stroke (width 0) (type default))
@@
     (stroke (width 0) (type default))
   )
+  (wire (pts (xy 496.57 106.68) (xy 496.57 120.65))
+    (stroke (width 0) (type default))
+  )
   (wire (pts (xy 144.78 130.81) (xy 154.94 130.81))
     (stroke (width 0) (type default))
@@
     (stroke (width 0) (type default))
   )
+  (wire (pts (xy 486.41 120.65) (xy 496.57 120.65))
+    (stroke (width 0) (type default))
+  )
   (wire (pts (xy 280.67 351.79) (xy 280.67 379.73))
     (stroke (width 0) (type default))
@@
     )
   )
+  (symbol (lib_id "Device:R") (at 496.57 102.87 0) (unit 1)
+    (in_bom yes) (on_board yes) (dnp no) (fields_autoplaced)
+    (property "Reference" "R66" (at 499.11 101.6 0)
+      (effects (font (size 1.27 1.27)) (justify left))
+    )
+    (property "Value" "5.1k" (at 499.11 104.14 0)
+      (effects (font (size 1.27 1.27)) (justify left))
+    )
+    (property "Footprint" "Resistor_SMD:R_0603_1608Metric" (at 494.792 102.87 90)
+      (effects (font (size 1.27 1.27)) hide)
+    )
+    (property "Datasheet" "~" (at 496.57 102.87 0)
+      (effects (font (size 1.27 1.27)) hide)
+    )
+    (pin "1")
+    (pin "2")
+    (instances
+      (project "MecProInverter"
+        (path "/c9071429-8b0d-45bf-aa6d-71cc2b7f068c/87c5d68c-a194-45d1-987f-2b491b6ac1ab"
+          (reference "R66") (unit 1)
+        )
+      )
+    )
+  )
   (symbol (lib_id "power:+3.3V") (at 369.57 52.07 0) (unit 1)
     (in_bom yes) (on_board yes) (dnp no) (fields_autoplaced)
@@
         )
       )
+    )
+  )
+  (symbol (lib_id "Device:R") (at 486.41 102.87 0) (unit 1)
+    (in_bom yes) (on_board yes) (dnp no)
+    (property "Reference" "R67" (at 490.22 101.6 0)
+      (effects (font (size 1.27 1.27)))
+    )
+    (property "Value" "5.1k" (at 488.95 104.14 0)
+      (effects (font (size 1.27 1.27)))
+    )
+    (property "Footprint" "Resistor_SMD:R_0603_1608Metric" (at 484.632 102.87 90)
+      (effects (font (size 1.27 1.27)) hide)
+    )
+    (property "Datasheet" "~" (at 486.41 102.87 0)
+      (effects (font (size 1.27 1.27)) hide)
+    )
+    (pin "1")
+    (pin "2")
+    (instances
+      (project "MecProInverter"
+        (path "/c9071429-8b0d-45bf-aa6d-71cc2b7f068c/87c5d68c-a194-45d1-987f-2b491b6ac1ab"
+          (reference "R67") (unit 1)
+        )
+      )

Commit message: Electronic
Layout begin
Connections:
- net +3.3V: now also C35.1, U2.12 (PIN), U2.13 (SPD), U2.14 (VDD2)
- net USB_DN renamed USB_N
- net USB_DP renamed USB_P
Changed lines of the file:
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@@
   (junction (at 377.19 120.65) (diameter 0) (color 0 0 0 0)
   )
+  (junction (at 353.06 54.61) (diameter 0) (color 0 0 0 0)
+  )
   (junction (at 389.89 74.93) (diameter 0) (color 0 0 0 0)
   )
@@
   )
   (junction (at 252.73 358.14) (diameter 0) (color 0 0 0 0)
+  )
+  (junction (at 353.06 62.23) (diameter 0) (color 0 0 0 0)
   )
   (junction (at 476.25 160.02) (diameter 0) (color 0 0 0 0)
@@
     (stroke (width 0) (type default))
   )
+  (wire (pts (xy 353.06 54.61) (xy 353.06 62.23))
+    (stroke (width 0) (type default))
+  )
   (wire (pts (xy 151.13 135.89) (xy 151.13 137.16))
     (stroke (width 0) (type default))
@@
     (stroke (width 0) (type default))
   )
-  (wire (pts (xy 328.93 69.85) (xy 359.41 69.85))
-    (stroke (width 0) (type default))
-  )
   (wire (pts (xy 533.4 67.31) (xy 525.78 67.31))
     (stroke (width 0) (type default))
@@
     (stroke (width 0) (type default))
   )
+  (wire (pts (xy 353.06 54.61) (xy 339.09 54.61))
+    (stroke (width 0) (type default))
+  )
   (wire (pts (xy 90.17 367.03) (xy 90.17 365.76))
     (stroke (width 0) (type default))
@@
     (stroke (width 0) (type default))
   )
-  (wire (pts (xy 369.57 54.61) (xy 339.09 54.61))
+  (wire (pts (xy 369.57 54.61) (xy 353.06 54.61))
     (stroke (width 0) (type default))
   )
@@
     (stroke (width 0) (type default))
   )
-  (wire (pts (xy 328.93 72.39) (xy 359.41 72.39))
-    (stroke (width 0) (type default))
-  )
   (wire (pts (xy 561.34 80.01) (xy 561.34 120.65))
     (stroke (width 0) (type default))
@@
     (stroke (width 0) (type default))
   )
+  (wire (pts (xy 321.31 72.39) (xy 359.41 72.39))
+    (stroke (width 0) (type default))
+  )
   (wire (pts (xy 115.57 110.49) (xy 120.65 110.49))
     (stroke (width 0) (type default))
@@
   )
   (wire (pts (xy 486.41 120.65) (xy 496.57 120.65))
+    (stroke (width 0) (type default))
+  )
+  (wire (pts (xy 321.31 69.85) (xy 359.41 69.85))
     (stroke (width 0) (type default))
   )
@@
     (effects (font (size 1.27 1.27)) (justify left bottom))
   )
-  (label "USB_DP" (at 328.93 69.85 0) (fields_autoplaced)
+  (label "USB_P" (at 321.31 69.85 0) (fields_autoplaced)
     (effects (font (size 1.27 1.27)) (justify left bottom))
   )
@@
     (effects (font (size 1.27 1.27)) (justify right bottom))
   )
-  (label "USB_DN" (at 328.93 72.39 0) (fields_autoplaced)
+  (label "USB_N" (at 321.31 72.39 0) (fields_autoplaced)
     (effects (font (size 1.27 1.27)) (justify left bottom))
   )
@@
     (effects (font (size 1.27 1.27)) (justify left bottom))
   )
-  (label "USB_DP" (at 196.85 92.71 0) (fields_autoplaced)
+  (label "USB_P" (at 196.85 92.71 0) (fields_autoplaced)
     (effects (font (size 1.27 1.27)) (justify left bottom))
   )
@@
     (effects (font (size 1.27 1.27)) (justify left bottom))
   )
-  (label "USB_DN" (at 196.85 90.17 0) (fields_autoplaced)
-    (effects (font (size 1.27 1.27)) (justify left bottom))
-  )
+  (label "USB_N" (at 196.85 90.17 0) (fields_autoplaced)
+    (effects (font (size 1.27 1.27)) (justify left bottom))
+  )
