File: electronic/MecProInverter/control.kicad_sch (KiCad schematic)
At the start: 89 parts, among them J3 ISO_Data, J5 Display, J6 MAX312820, J7 Test, Q1 DMN3404L, SW1 PTS645SM95SMTR92LFS, SW2 PTS645SM95SMTR92LFS, SW3 PTS645SM95SMTR92LFS, U1 ESP32-S3-MINI-1-N8, U12 TEA1-0505HI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

Commit message: Electronic
PCB buy!!!
Parts:
- C37: value 10uF -> 22uF
- Fan1, Fan2, J3, J5, J6, J7: now left out of the parts list
- R38: value 165 -> 121
- R49, R50, R51, R52: value 180 -> 121
Changed lines of the file:
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@@
       (effects (font (size 1.27 1.27)))
     )
-    (property "Value" "180" (at 271.78 341.63 90)
+    (property "Value" "121" (at 271.78 341.63 90)
       (effects (font (size 1.27 1.27)))
     )
@@
       (effects (font (size 1.27 1.27)))
     )
-    (property "Value" "180" (at 271.78 346.71 90)
+    (property "Value" "121" (at 271.78 346.71 90)
       (effects (font (size 1.27 1.27)))
     )
@@
       (effects (font (size 1.27 1.27)))
     )
-    (property "Value" "165" (at 384.81 203.2 90)
+    (property "Value" "121" (at 384.81 203.2 90)
       (effects (font (size 1.27 1.27)))
     )
@@
   )
   (symbol (lib_id "dk_Rectangular-Connectors-Headers-Male-Pins:0022232031") (at 532.13 170.18 180) (unit 1)
-    (in_bom yes) (on_board yes) (dnp no)
+    (in_bom no) (on_board yes) (dnp no)
     (property "Reference" "Fan2" (at 530.86 166.37 0)
       (effects (font (size 1.27 1.27)) (justify left))
@@
   )
   (symbol (lib_id "Connector_Generic:Conn_01x03") (at 215.9 257.81 0) (mirror y) (unit 1)
-    (in_bom yes) (on_board yes) (dnp no) (fields_autoplaced)
+    (in_bom no) (on_board yes) (dnp no) (fields_autoplaced)
     (property "Reference" "J6" (at 215.9 248.92 0)
       (effects (font (size 1.27 1.27)))
@@
       (effects (font (size 1.27 1.27)))
     )
-    (property "Value" "180" (at 280.67 344.17 90)
+    (property "Value" "121" (at 280.67 344.17 90)
       (effects (font (size 1.27 1.27)))
     )
@@
       (effects (font (size 1.27 1.27)) (justify left))
     )
-    (property "Value" "10uF" (at 520.7 86.36 0)
+    (property "Value" "22uF" (at 520.7 86.36 0)
       (effects (font (size 1.27 1.27)) (justify left))
     )
@@
   )
   (symbol (lib_id "Connector_Generic:Conn_01x08") (at 523.24 309.88 0) (unit 1)
-    (in_bom yes) (on_board yes) (dnp no) (fields_autoplaced)
+    (in_bom no) (on_board yes) (dnp no) (fields_autoplaced)
     (property "Reference" "J5" (at 525.78 309.88 0)
       (effects (font (size 1.27 1.27)) (justify left))
@@
   )
   (symbol (lib_id "dk_Rectangular-Connectors-Headers-Male-Pins:0022232031") (at 509.27 170.18 180) (unit 1)
-    (in_bom yes) (on_board yes) (dnp no)
+    (in_bom no) (on_board yes) (dnp no)
     (property "Reference" "Fan1" (at 508 166.37 0)
       (effects (font (size 1.27 1.27)) (justify left))
@@
   )
   (symbol (lib_id "Connector_Generic:Conn_01x11") (at 48.26 234.95 180) (unit 1)
-    (in_bom yes) (on_board yes) (dnp no) (fields_autoplaced)
+    (in_bom no) (on_board yes) (dnp no) (fields_autoplaced)
     (property "Reference" "J7" (at 48.26 215.9 0)
       (effects (font (size 1.27 1.27)))
@@
   )
   (symbol (lib_id "Connector:Screw_Terminal_01x06") (at 292.1 344.17 0) (unit 1)
-    (in_bom yes) (on_board yes) (dnp no) (fields_autoplaced)
+    (in_bom no) (on_board yes) (dnp no) (fields_autoplaced)
     (property "Reference" "J3" (at 294.64 344.17 0)
       (effects (font (size 1.27 1.27)) (justify left))
@@
       (effects (font (size 1.27 1.27)))
     )
-    (property "Value" "180" (at 280.67 339.09 90)
+    (property "Value" "121" (at 280.67 339.09 90)
       (effects (font (size 1.27 1.27)))
     )
