File: electronic/MecProInverter/control.kicad_sch (KiCad schematic)
At the start: 89 parts, among them J3 ISO_Data, J5 Display, J6 MAX312820, J7 Test, Q1 DMN3404L, SW1 PTS645SM95SMTR92LFS, SW2 PTS645SM95SMTR92LFS, SW3 PTS645SM95SMTR92LFS, U1 ESP32-S3-MINI-1-N8, U12 TEA1-0505HI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

Commit message: Software
Added Pinout
Created arduino Hardware Test
Connections:
- net +3.3V: now also C5.1
- net RGBLED: no longer C5.1
Changed lines of the file:
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@@
   (junction (at 90.17 339.09) (diameter 0) (color 0 0 0 0)
   )
-  (junction (at 391.16 308.61) (diameter 0) (color 0 0 0 0)
-  )
   (junction (at 90.17 374.65) (diameter 0) (color 0 0 0 0)
   )
@@
   )
   (junction (at 389.89 120.65) (diameter 0) (color 0 0 0 0)
+  )
+  (junction (at 408.94 297.18) (diameter 0) (color 0 0 0 0)
   )
   (junction (at 528.32 54.61) (diameter 0) (color 0 0 0 0)
@@
     (stroke (width 0) (type default))
   )
+  (wire (pts (xy 391.16 309.88) (xy 391.16 297.18))
+    (stroke (width 0) (type default))
+  )
   (wire (pts (xy 243.84 374.65) (xy 252.73 374.65))
     (stroke (width 0) (type default))
@@
     (stroke (width 0) (type default))
   )
+  (wire (pts (xy 391.16 297.18) (xy 408.94 297.18))
+    (stroke (width 0) (type default))
+  )
   (wire (pts (xy 104.14 101.6) (xy 104.14 97.79))
     (stroke (width 0) (type default))
@@
     (stroke (width 0) (type default))
   )
-  (wire (pts (xy 408.94 295.91) (xy 408.94 300.99))
+  (wire (pts (xy 408.94 295.91) (xy 408.94 297.18))
     (stroke (width 0) (type default))
   )
@@
     (stroke (width 0) (type default))
   )
-  (wire (pts (xy 382.27 308.61) (xy 391.16 308.61))
-    (stroke (width 0) (type default))
-  )
   (wire (pts (xy 148.59 133.35) (xy 148.59 134.62))
     (stroke (width 0) (type default))
@@
     (stroke (width 0) (type default))
   )
+  (wire (pts (xy 408.94 297.18) (xy 408.94 300.99))
+    (stroke (width 0) (type default))
+  )
   (wire (pts (xy 196.85 107.95) (xy 185.42 107.95))
     (stroke (width 0) (type default))
@@
     (stroke (width 0) (type default))
   )
-  (wire (pts (xy 391.16 308.61) (xy 391.16 309.88))
-    (stroke (width 0) (type default))
-  )
   (wire (pts (xy 63.5 224.79) (xy 53.34 224.79))
     (stroke (width 0) (type default))
@@
     (stroke (width 0) (type default))
   )
-  (wire (pts (xy 391.16 308.61) (xy 401.32 308.61))
-    (stroke (width 0) (type default))
-  )
+  (wire (pts (xy 382.27 308.61) (xy 401.32 308.61))
+    (stroke (width 0) (type default))
+  )
